Commit message: 修改urdf模型

File: legged_gym/resources/robots/black/urdf/black_description.urdf (robot description, URDF)
Before this commit: robot black_description, 19 links, 18 joints
Links:
- link FL_calf: mass 0.25559 -> 0.24861
- link FL_thigh: mass 0.83909 -> 0.91168
- link FR_calf: mass 0.25559 -> 0.24861
- link FR_thigh: mass 0.84232 -> 0.91491
- link RL_calf: mass 0.25559 -> 0.24861
- link RL_thigh: mass 0.83909 -> 0.91168
- link RR_calf: mass 0.25559 -> 0.24861
- link RR_thigh: mass 0.84232 -> 0.91491
- link trunk: mass 5.722 -> 5.7042
Joints:
- joint FL_foot_fixed: origin xyz=0 -0.0078843 -0.25749 rpy=0 0 0 -> xyz=0 -0.013803 -0.24433 rpy=0 0 0
- joint FR_foot_fixed: origin xyz=0 0.0078843 -0.25749 rpy=0 0 0 -> xyz=0 0.013803 -0.24433 rpy=0 0 0
- joint RL_foot_fixed: origin xyz=0 -0.0078843 -0.25749 rpy=0 0 0 -> xyz=0 -0.013803 -0.24433 rpy=0 0 0
- joint RR_foot_fixed: origin xyz=0 0.0078843 -0.25749 rpy=0 0 0 -> xyz=0 0.013803 -0.24433 rpy=0 0 0

Commit message: 修复指令课程学习bug & checkpoint

File: legged_gym/resources/robots/black/urdf/black_description.urdf (robot description, URDF)
Before this commit: robot black_description, 19 links, 18 joints
Joints:
- joint FL_calf_joint: limit lower=-10 upper=10 effort=20 velocity=25 -> lower=-2.5 upper=-0.85 effort=20 velocity=25
- joint FL_hip_joint: limit lower=-10 upper=10 effort=20 velocity=25 -> lower=-0.5 upper=0.5 effort=20 velocity=25
- joint FL_thigh_joint: limit lower=-10 upper=10 effort=20 velocity=25 -> lower=-1.2 upper=1.6 effort=20 velocity=25
- joint FR_calf_joint: limit lower=-10 upper=10 effort=20 velocity=25 -> lower=0.85 upper=2.5 effort=20 velocity=25
- joint FR_hip_joint: limit lower=-10 upper=10 effort=20 velocity=25 -> lower=-0.5 upper=0.5 effort=20 velocity=25
- joint FR_thigh_joint: limit lower=-10 upper=10 effort=20 velocity=25 -> lower=-1.6 upper=1.2 effort=20 velocity=25
- joint RL_calf_joint: limit lower=-10 upper=10 effort=20 velocity=25 -> lower=-2.5 upper=-0.85 effort=20 velocity=25
- joint RL_hip_joint: limit lower=-10 upper=10 effort=20 velocity=25 -> lower=-0.5 upper=0.5 effort=20 velocity=25
- joint RL_thigh_joint: limit lower=-10 upper=10 effort=20 velocity=25 -> lower=-1.2 upper=1.6 effort=20 velocity=25
- joint RR_calf_joint: limit lower=-10 upper=10 effort=20 velocity=25 -> lower=0.85 upper=2.5 effort=20 velocity=25
- joint RR_hip_joint: limit lower=-10 upper=10 effort=20 velocity=25 -> lower=-0.5 upper=0.5 effort=20 velocity=25
- joint RR_thigh_joint: limit lower=-10 upper=10 effort=20 velocity=25 -> lower=-1.6 upper=1.2 effort=20 velocity=25
