Commit message: 修改urdf

File: legged_gym/resources/robots/black/black_description.urdf (robot description, URDF)
Before this commit: robot black_description, 19 links, 18 joints
Links:
- link FL_calf: geometry collision cylinder length=0.04 radius=0.02; collision cylinder length=0.05 radius=0.014
- link FL_foot: geometry collision sphere radius=0.02; visual sphere radius=0.02
- link FL_thigh: geometry collision box size=0.035 0.05 0.205; visual mesh filename=meshes/FL_thigh.STL
- link FR_calf: geometry collision cylinder length=0.04 radius=0.02; collision cylinder length=0.05 radius=0.014
- link FR_foot: geometry collision sphere radius=0.02; visual sphere radius=0.02
- link FR_thigh: geometry collision box size=0.035 0.05 0.205; visual mesh filename=meshes/FR_thigh.STL
- link RL_calf: geometry collision cylinder length=0.04 radius=0.02; collision cylinder length=0.05 radius=0.014
- link RL_foot: geometry collision sphere radius=0.02; visual sphere radius=0.02
- link RL_thigh: geometry collision box size=0.035 0.05 0.205; visual mesh filename=meshes/RL_thigh.STL
- link RR_calf: geometry collision cylinder length=0.04 radius=0.02; collision cylinder length=0.05 radius=0.014
- link RR_foot: geometry collision sphere radius=0.02; visual sphere radius=0.02
- link RR_thigh: geometry collision box size=0.035 0.05 0.205; visual mesh filename=meshes/RR_thigh.STL

Commit message: 修改urdf

File: legged_gym/resources/robots/black/black_description.urdf (robot description, URDF)
Before this commit: robot black_description, 19 links, 18 joints
Links:
- added link d435_link, mass 0.072; visual mesh filename=meshes/d435.stl
- link trunk: geometry collision box size=0.01 0.09 0.14; collision box size=0.145 0.07 0.01
Joints:
- added joint d435_joint: type fixed, parent trunk, child d435_link, origin xyz=0.225 0 0.028 rpy=0 0 0

File: legged_gym/resources/robots/black_with_arm/urdf/black_with_arm.urdf (robot description, URDF)
Before this commit: robot black_with_arm_draft, 25 links, 24 joints
Links:
- added link d435_link, mass 0.072; visual mesh filename=../meshes_black/d435.stl
- link FL_calf: geometry collision cylinder length=0.04 radius=0.02; collision cylinder length=0.05 radius=0.014
- link FL_foot: geometry collision sphere radius=0.02; visual sphere radius=0.02
- link FL_hip: geometry collision cylinder length=0.11 radius=0.052; visual mesh filename=../meshes_black/FL_hip.STL
- link FL_thigh: geometry collision box size=0.035 0.05 0.205; visual mesh filename=../meshes_black/FL_thigh.STL
- link FR_calf: geometry collision cylinder length=0.04 radius=0.02; collision cylinder length=0.05 radius=0.014
- link FR_foot: geometry collision sphere radius=0.02; visual sphere radius=0.02
- link FR_hip: geometry collision cylinder length=0.11 radius=0.052; visual mesh filename=../meshes_black/FR_hip.STL
- link FR_thigh: geometry collision box size=0.035 0.05 0.205; visual mesh filename=../meshes_black/FR_thigh.STL
- link RL_calf: geometry collision cylinder length=0.04 radius=0.02; collision cylinder length=0.05 radius=0.014
- link RL_foot: geometry collision sphere radius=0.02; visual sphere radius=0.02
- link RL_hip: geometry collision cylinder length=0.11 radius=0.052; visual mesh filename=../meshes_black/RL_hip.STL
- link RL_thigh: geometry collision box size=0.035 0.05 0.205; visual mesh filename=../meshes_black/RL_thigh.STL
- link RR_calf: geometry collision cylinder length=0.04 radius=0.02; collision cylinder length=0.05 radius=0.014
- link RR_foot: geometry collision sphere radius=0.02; visual sphere radius=0.02
- link RR_hip: geometry collision cylinder length=0.11 radius=0.052; visual mesh filename=../meshes_black/RR_hip.STL
- link RR_thigh: geometry collision box size=0.035 0.05 0.205; visual mesh filename=../meshes_black/RR_thigh.STL
- link trunk: geometry collision box size=0.01 0.09 0.14; collision box size=0.145 0.07 0.01
Joints:
- added joint d435_joint: type fixed, parent trunk, child d435_link, origin xyz=0.225 0 0.028 rpy=0 0 0

File: legged_gym/resources/robots/black_with_arm/urdf/black_with_arm_train.urdf (robot description, URDF)
Before this commit: robot black_with_arm_train, 25 links, 24 joints
Links:
- added link d435_link, mass 0.072; visual mesh filename=../meshes_black/d435.stl
- link FL_calf: geometry collision cylinder length=0.04 radius=0.02; collision cylinder length=0.05 radius=0.014
- link FL_foot: geometry collision sphere radius=0.02; visual sphere radius=0.02
- link FL_hip: geometry collision cylinder length=0.11 radius=0.052; visual mesh filename=../meshes_black/FL_hip.STL
- link FL_thigh: geometry collision box size=0.035 0.05 0.205; visual mesh filename=../meshes_black/FL_thigh.STL
- link FR_calf: geometry collision cylinder length=0.04 radius=0.02; collision cylinder length=0.05 radius=0.014
- link FR_foot: geometry collision sphere radius=0.02; visual sphere radius=0.02
- link FR_hip: geometry collision cylinder length=0.11 radius=0.052; visual mesh filename=../meshes_black/FR_hip.STL
- link FR_thigh: geometry collision box size=0.035 0.05 0.205; visual mesh filename=../meshes_black/FR_thigh.STL
- link RL_calf: geometry collision cylinder length=0.04 radius=0.02; collision cylinder length=0.05 radius=0.014
- link RL_foot: geometry collision sphere radius=0.02; visual sphere radius=0.02
- link RL_hip: geometry collision cylinder length=0.11 radius=0.052; visual mesh filename=../meshes_black/RL_hip.STL
- link RL_thigh: geometry collision box size=0.035 0.05 0.205; visual mesh filename=../meshes_black/RL_thigh.STL
- link RR_calf: geometry collision cylinder length=0.04 radius=0.02; collision cylinder length=0.05 radius=0.014
- link RR_foot: geometry collision sphere radius=0.02; visual sphere radius=0.02
- link RR_hip: geometry collision cylinder length=0.11 radius=0.052; visual mesh filename=../meshes_black/RR_hip.STL
- link RR_thigh: geometry collision box size=0.035 0.05 0.205; visual mesh filename=../meshes_black/RR_thigh.STL
- link trunk: geometry collision box size=0.01 0.09 0.14; collision box size=0.145 0.07 0.01
Joints:
- added joint d435_joint: type fixed, parent trunk, child d435_link, origin xyz=0.225 0 0.028 rpy=0 0 0
