Commit message: 更新urdf,微调奖励,新增轮速规划奖励

File: legged_gym/resources/robots/blackW/blackW_description.urdf (robot description, URDF)
Before this commit: robot blackW, 20 links, 19 joints
Links:
- link FL_calf: mass 0.24861 -> 0.6311814
- link FL_foot: mass 2.7328 -> 1.4862602; geometry collision cylinder length=0.049 radius=0.103; visual mesh filename=meshes/FL_foot.STL
- link FL_hip: mass 0.60559 -> 0.6055878; geometry collision cylinder length=0.06 radius=0.052; visual mesh filename=meshes/FL_hip.STL
- link FL_thigh: mass 0.91168 -> 0.9116849; geometry collision box size=0.035 0.05 0.205; collision cylinder length=0.035 radius=0.052
- link FR_calf: mass 0.24861 -> 0.6311813
- link FR_foot: mass 2.7328 -> 1.4862603; geometry collision cylinder length=0.049 radius=0.103; visual mesh filename=meshes/FR_foot.STL
- link FR_hip: mass 0.60559 -> 0.6055878; geometry collision cylinder length=0.06 radius=0.052; visual mesh filename=meshes/FR_hip.STL
- link FR_thigh: mass 0.91491 -> 0.9149128; geometry collision box size=0.035 0.05 0.205; collision cylinder length=0.035 radius=0.052
- link RL_calf: mass 0.24861 -> 0.6311814
- link RL_foot: mass 2.7328 -> 1.4862602; geometry collision cylinder length=0.049 radius=0.103; visual mesh filename=meshes/RL_foot.STL
- link RL_hip: mass 0.60559 -> 0.6055878; geometry collision cylinder length=0.06 radius=0.052; visual mesh filename=meshes/RL_hip.STL
- link RL_thigh: mass 0.91168 -> 0.9116849; geometry collision box size=0.035 0.05 0.205; collision cylinder length=0.035 radius=0.052
- link RR_calf: mass 0.24861 -> 0.6311815
- link RR_foot: mass 2.7328 -> 1.4862602; geometry collision cylinder length=0.049 radius=0.103; visual mesh filename=meshes/RR_foot.STL
- link RR_hip: mass 0.60559 -> 0.6055878; geometry collision cylinder length=0.06 radius=0.052; visual mesh filename=meshes/RR_hip.STL
- link RR_thigh: mass 0.91491 -> 0.9149128; geometry collision box size=0.035 0.05 0.205; collision cylinder length=0.035 radius=0.052
- link trunk: mass 5.766 -> 5.7659525
